Commit message: Revert "limo_circle_sim: replace LIMO mesh visuals with primitives (Option C)"
This reverts commit 2f7dc054379de168cd47acdad725e1af4b3e292f.

File: ros2/limo_circle_sim/urdf/limo_four_diff.xacro (robot description, xacro)
@@ -23,22 +23,17 @@
   </joint>
     <!-- Base link -->
-    <!-- Visual replaced with a simple box (was: limo_base.dae) so gzclient/rviz
-         don't have to render a 50 MB DAE per robot. UTM/M1 has no GPU acceleration
-         for Linux so software rendering of large meshes OOM-kills the viewer. -->
     <link name="base_link">
         <visual>
-            <origin xyz="0 0 0" rpy="0 0 0" />
+            <origin xyz="0 0 -0.15" rpy="0 0 1.57" />
             <geometry>
-                <box size="${base_x_size} ${base_y_size} ${base_z_size}"/>
+                <mesh filename="file://$(find limo_circle_sim)/meshes/limo_base.dae" scale="1 1 1"/>
             </geometry>
-            <material name="limo_yellow">
-                <color rgba="1.0 0.85 0.1 1"/>
-            </material>
         </visual>
         <collision>
+            <!--origin xyz="0 0 -0.15" rpy="0 0 1.57" /-->
             <origin xyz="0 0 0" rpy="0 0 0" />
-            <geometry>
-                <box size="${base_x_size} ${base_y_size} ${base_z_size}"/>
-            </geometry>
+          <geometry>
+              <box size="${base_x_size} ${base_y_size} ${base_z_size}"/>
+          </geometry>
         </collision>
     </link>

File: ros2/limo_circle_sim/urdf/limo_xacro.xacro (robot description, xacro)
@@ -8,14 +8,9 @@
                 <inertia ixx="0.01055" ixy="0" ixz="0" iyy="0.00075" iyz="0" izz="0.01055" />
             </inertial>
-            <!-- Visual replaced with cylinder primitive (was: limo_wheel.dae)
-                 to skip 11 MB DAE per wheel × 4 wheels × N robots. -->
             <visual>
-                <origin xyz="0 ${wheel_length/2} 0" rpy="1.57 0 0" />
+                <origin xyz="0 0 0" rpy="0 0 0" />
                 <geometry>
-                    <cylinder length="${wheel_length}" radius="${wheel_radius}" />
+                    <mesh filename="file://$(find limo_circle_sim)/meshes/limo_wheel.dae" />
                 </geometry>
-                <material name="wheel_black">
-                    <color rgba="0.1 0.1 0.1 1"/>
-                </material>
             </visual>
             <collision>
