Commit message: limo_circle_sim: replace LIMO mesh visuals with primitives (Option C)
Even with 10 GB VM RAM, gzclient gets OOM-killed on M1 UTM because
UTM has no GPU passthrough for Linux — software OGRE rendering of
the 50 MB limo_base.dae × N robots blows up. Same story for rviz2.

Replace:
- base_link visual: <mesh limo_base.dae> → <box 0.13 x 0.12 x 0.1>
  (matches existing collision shape; coloured limo-yellow)
- wheel visual:     <mesh limo_wheel.dae> → <cylinder r=0.045 l=0.045>
  (matches existing collision shape; coloured black)

Drop the now-unused .dae files (~61 MB) and the unused
limo_steering_hinge.xacro (Ackermann variant, never included by our
limo_four_diff.xacro path).

Physics is unchanged — the diff_drive plugin only cares about
collisions, which were already box+cylinder primitives. Looks
Lego-y but renders instantly even under software GL.

Co-Authored-By: Claude Opus 4.7 <noreply@anthropic.com>

File: ros2/limo_circle_sim/urdf/limo_four_diff.xacro (robot description, xacro)
@@ -23,17 +23,22 @@
   </joint>
     <!-- Base link -->
+    <!-- Visual replaced with a simple box (was: limo_base.dae) so gzclient/rviz
+         don't have to render a 50 MB DAE per robot. UTM/M1 has no GPU acceleration
+         for Linux so software rendering of large meshes OOM-kills the viewer. -->
     <link name="base_link">
         <visual>
-            <origin xyz="0 0 -0.15" rpy="0 0 1.57" />
+            <origin xyz="0 0 0" rpy="0 0 0" />
             <geometry>
-                <mesh filename="file://$(find limo_circle_sim)/meshes/limo_base.dae" scale="1 1 1"/>
+                <box size="${base_x_size} ${base_y_size} ${base_z_size}"/>
             </geometry>
+            <material name="limo_yellow">
+                <color rgba="1.0 0.85 0.1 1"/>
+            </material>
         </visual>
         <collision>
-            <!--origin xyz="0 0 -0.15" rpy="0 0 1.57" /-->
             <origin xyz="0 0 0" rpy="0 0 0" />
-          <geometry>
-              <box size="${base_x_size} ${base_y_size} ${base_z_size}"/>
-          </geometry>
+            <geometry>
+                <box size="${base_x_size} ${base_y_size} ${base_z_size}"/>
+            </geometry>
         </collision>
     </link>

File: ros2/limo_circle_sim/urdf/limo_xacro.xacro (robot description, xacro)
@@ -8,9 +8,14 @@
                 <inertia ixx="0.01055" ixy="0" ixz="0" iyy="0.00075" iyz="0" izz="0.01055" />
             </inertial>
+            <!-- Visual replaced with cylinder primitive (was: limo_wheel.dae)
+                 to skip 11 MB DAE per wheel × 4 wheels × N robots. -->
             <visual>
-                <origin xyz="0 0 0" rpy="0 0 0" />
+                <origin xyz="0 ${wheel_length/2} 0" rpy="1.57 0 0" />
                 <geometry>
-                    <mesh filename="file://$(find limo_circle_sim)/meshes/limo_wheel.dae" />
+                    <cylinder length="${wheel_length}" radius="${wheel_radius}" />
                 </geometry>
+                <material name="wheel_black">
+                    <color rgba="0.1 0.1 0.1 1"/>
+                </material>
             </visual>
             <collision>

Commit message: limo_circle_sim: bundle .dae meshes + use_real_meshes launch arg; v2 first in README
Two changes prompted by user feedback after polishing the README:

1. **Real LIMO meshes are bundled again, opt-in via launch arg.**
   Restored ros2/limo_circle_sim/meshes/limo_base.dae (~52 MB) and
   limo_wheel.dae (~11 MB) from f12a5a4. Wrapped each `<visual>` block
   in urdf/limo_four_diff.xacro (base_link) and urdf/limo_xacro.xacro
   (wheel macro) in `<xacro:if value="$(arg use_real_meshes)">` /
   `<xacro:unless>` so the same URDF emits either the mesh visual or
   the primitive box/cylinder depending on the xacro arg.

   New launch arg `use_real_meshes` (default `false`) plumbs to xacro
   via the Command in `_spawn_one`. Default keeps the M1-UTM-friendly
   primitive visuals; `use_real_meshes:=true` opts into photorealistic
   AgileX meshes for hosts with real GPU acceleration.

   Replaces the previous "revert this commit to get meshes back"
   workflow — users just pass a flag now. Collision geometry stays
   primitive in both modes so physics is unchanged.

2. **README reordered to lead with policy_v2 / hallway_node.** That's
   the current default policy for new demos, so the showcase section
   now puts hallway_node as "Option A" with circle_node as "Option B
   (alternative)". Intro bullet order flipped to match. M1-UTM
   callout reworded to explain why `use_real_meshes` defaults false,
   pointing at the launch arg rather than git revert instructions.

   Mesh-switching section is now a 2-line table + one bash snippet
   instead of the previous two-option git-surgery walkthrough.

Co-Authored-By: Claude Opus 4.7 <noreply@anthropic.com>

File: ros2/limo_circle_sim/urdf/limo_four_diff.xacro (robot description, xacro)
@@ -2,4 +2,12 @@
 <robot name="limo_four_diff" xmlns:xacro="http://ros.org/wiki/xacro">
     <xacro:arg name="robot_namespace" default="/" />
+    <!-- use_real_meshes=true → load the original AgileX .dae visuals
+                              (52 MB body + 11 MB wheel × 4 per robot).
+                              Looks nice on a host with real GPU.
+         use_real_meshes=false → render the body as a yellow box and the
+                                 wheels as black cylinders. ~1 KB per robot,
+                                 survives software OpenGL (UTM on M1 etc.).
+         Collision geometry is the same in both cases. -->
+    <xacro:arg name="use_real_meshes" default="false" />
     <xacro:include filename="$(find limo_circle_sim)/urdf/limo_xacro.xacro" />
     <xacro:include filename="$(find limo_circle_sim)/urdf/limo_four_diff.gazebo" />
@@ -23,17 +31,24 @@
   </joint>
     <!-- Base link -->
-    <!-- Visual replaced with a simple box (was: limo_base.dae) so gzclient/rviz
-         don't have to render a 50 MB DAE per robot. UTM/M1 has no GPU acceleration
-         for Linux so software rendering of large meshes OOM-kills the viewer. -->
     <link name="base_link">
-        <visual>
-            <origin xyz="0 0 0" rpy="0 0 0" />
-            <geometry>
-                <box size="${base_x_size} ${base_y_size} ${base_z_size}"/>
-            </geometry>
-            <material name="limo_yellow">
-                <color rgba="1.0 0.85 0.1 1"/>
-            </material>
-        </visual>
+        <xacro:if value="$(arg use_real_meshes)">
+            <visual>
+                <origin xyz="0 0 -0.15" rpy="0 0 1.57" />
+                <geometry>
+                    <mesh filename="file://$(find limo_circle_sim)/meshes/limo_base.dae" scale="1 1 1"/>
+                </geometry>
+            </visual>
+        </xacro:if>
+        <xacro:unless value="$(arg use_real_meshes)">
+            <visual>
+                <origin xyz="0 0 0" rpy="0 0 0" />
+                <geometry>
+                    <box size="${base_x_size} ${base_y_size} ${base_z_size}"/>
+                </geometry>
+                <material name="limo_yellow">
+                    <color rgba="1.0 0.85 0.1 1"/>
+                </material>
+            </visual>
+        </xacro:unless>
         <collision>
             <origin xyz="0 0 0" rpy="0 0 0" />

File: ros2/limo_circle_sim/urdf/limo_xacro.xacro (robot description, xacro)
@@ -1,4 +1,6 @@
 <?xml version="1.0"?>
 <robot name="limo_xacro" xmlns:xacro="http://ros.org/wiki/xacro">
+    <!-- use_real_meshes arg is declared on the top-level limo_four_diff.xacro
+         and inherited here. true → wheel mesh DAE, false → cylinder primitive. -->
     <xacro:macro name="limo_wheel" params="parent_prefix wheel_prefix reflect *joint_pose">
         <link name="${wheel_prefix}_wheel_link">
@@ -8,15 +10,23 @@
                 <inertia ixx="0.01055" ixy="0" ixz="0" iyy="0.00075" iyz="0" izz="0.01055" />
             </inertial>
-            <!-- Visual replaced with cylinder primitive (was: limo_wheel.dae)
-                 to skip 11 MB DAE per wheel × 4 wheels × N robots. -->
-            <visual>
-                <origin xyz="0 ${wheel_length/2} 0" rpy="1.57 0 0" />
-                <geometry>
-                    <cylinder length="${wheel_length}" radius="${wheel_radius}" />
-                </geometry>
-                <material name="wheel_black">
-                    <color rgba="0.1 0.1 0.1 1"/>
-                </material>
-            </visual>
+            <xacro:if value="$(arg use_real_meshes)">
+                <visual>
+                    <origin xyz="0 0 0" rpy="0 0 0" />
+                    <geometry>
+                        <mesh filename="file://$(find limo_circle_sim)/meshes/limo_wheel.dae" />
+                    </geometry>
+                </visual>
+            </xacro:if>
+            <xacro:unless value="$(arg use_real_meshes)">
+                <visual>
+                    <origin xyz="0 ${wheel_length/2} 0" rpy="1.57 0 0" />
+                    <geometry>
+                        <cylinder length="${wheel_length}" radius="${wheel_radius}" />
+                    </geometry>
+                    <material name="wheel_black">
+                        <color rgba="0.1 0.1 0.1 1"/>
+                    </material>
+                </visual>
+            </xacro:unless>
             <collision>
               <origin xyz="0 ${wheel_length/2} 0" rpy="1.57 0 0" />
